Commit message: add mpu6050 plugin and use to xacro and yaml

File: src/robot/robot_car_mecanum/urdf/robot_car.xacro (robot description, xacro)
@@ -21,4 +21,5 @@
       </xacro:if>
       <xacro:unless value="$(arg use_gazebo)">
+        <plugin>mpu6050_hw/MPU6050Hardware</plugin>
         <plugin>four_wheel_chassis_hw/FourWheelChassisHW</plugin>
         <!-- <plugin>mock_components/GenericSystem</plugin>
@@ -47,4 +48,36 @@
       <state_interface name="velocity"/>
     </joint>
+    <sensor name="mpu6050" state_interface_names="
+      mpu6050/accel_x,
+      mpu6050/accel_y,
+      mpu6050/accel_z,
+      mpu6050/gyro_x,
+      mpu6050/gyro_y,
+      mpu6050/gyro_z">
+      <state_interface name="accel_x">
+        <param name="interface_type">linear_acceleration</param>
+        <param name="unit">m/s²</param>
+      </state_interface>
+      <state_interface name="accel_y">
+        <param name="interface_type">linear_acceleration</param>
+        <param name="unit">m/s²</param>
+      </state_interface>
+      <state_interface name="accel_z">
+        <param name="interface_type">linear_acceleration</param>
+        <param name="unit">m/s²</param>
+      </state_interface>
+      <state_interface name="gyro_x">
+        <param name="interface_type">angular_velocity</param>
+        <param name="unit">rad/s</param>
+      </state_interface>
+      <state_interface name="gyro_y">
+        <param name="interface_type">angular_velocity</param>
+        <param name="unit">rad/s</param>
+      </state_interface>
+      <state_interface name="gyro_z">
+        <param name="interface_type">angular_velocity</param>
+        <param name="unit">rad/s</param>
+      </state_interface>
+    </sensor>
   </ros2_control>
 </robot>

File: src/robot/robot_desc/urdf/four_wheel_chassis.xacro (robot description, xacro)
@@ -120,3 +120,23 @@
     <origin xyz="0 0 0.05" rpy="0 0 0" />
   </joint>
+  <link name="imu">
+    <visual>
+      <geometry>
+        <box size="0.02 0.02 0.02"/>
+      </geometry>
+      <material name="gray">
+        <color rgba="0.5 0.5 0.5 1.0"/>
+      </material>
+    </visual>
+    <collision>
+      <geometry>
+        <box size="0.02 0.02 0.02"/>
+      </geometry>
+    </collision>
+  </link>
+  <joint name="imu_joint" type="fixed">
+    <parent link="base_link"/>
+    <child link="imu"/>
+    <origin xyz="0.1 0.0 0.05" rpy="0 0 0"/>
+  </joint>
 </robot>

Commit message: success add mpu6050

File: src/robot/robot_car_mecanum/urdf/robot_car.xacro (robot description, xacro)
@@ -7,5 +7,4 @@
   <xacro:include filename="$(find robot_desc)/urdf/four_wheel_chassis.xacro"/>
   <xacro:if value='$(arg use_gazebo)'>
-    <!-- Gazebo仿真特定配置 -->
     <gazebo>
       <plugin filename="gz_ros2_control-system" name="gz_ros2_control::GazeboSimROS2ControlPlugin">
@@ -14,6 +13,5 @@
     </gazebo>
   </xacro:if>
-  <!-- ros2_control配置 -->
-  <ros2_control name="CarSystem" type="system">
+  <ros2_control name="mecanum_wheels_chassis" type="system">
     <hardware>
       <xacro:if value="$(arg use_gazebo)">
@@ -21,5 +19,4 @@
       </xacro:if>
       <xacro:unless value="$(arg use_gazebo)">
-        <plugin>mpu6050_hw/MPU6050Hardware</plugin>
         <plugin>four_wheel_chassis_hw/FourWheelChassisHW</plugin>
         <!-- <plugin>mock_components/GenericSystem</plugin>
@@ -27,5 +24,4 @@
       </xacro:unless>
     </hardware>
-    <!-- 关节定义保持不变 -->
     <joint name="left_front_wheel_joint">
       <command_interface name="velocity"/>
@@ -48,36 +44,21 @@
       <state_interface name="velocity"/>
     </joint>
-    <sensor name="mpu6050" state_interface_names="
-      mpu6050/accel_x,
-      mpu6050/accel_y,
-      mpu6050/accel_z,
-      mpu6050/gyro_x,
-      mpu6050/gyro_y,
-      mpu6050/gyro_z">
-      <state_interface name="accel_x">
-        <param name="interface_type">linear_acceleration</param>
-        <param name="unit">m/s²</param>
-      </state_interface>
-      <state_interface name="accel_y">
-        <param name="interface_type">linear_acceleration</param>
-        <param name="unit">m/s²</param>
-      </state_interface>
-      <state_interface name="accel_z">
-        <param name="interface_type">linear_acceleration</param>
-        <param name="unit">m/s²</param>
-      </state_interface>
-      <state_interface name="gyro_x">
-        <param name="interface_type">angular_velocity</param>
-        <param name="unit">rad/s</param>
-      </state_interface>
-      <state_interface name="gyro_y">
-        <param name="interface_type">angular_velocity</param>
-        <param name="unit">rad/s</param>
-      </state_interface>
-      <state_interface name="gyro_z">
-        <param name="interface_type">angular_velocity</param>
-        <param name="unit">rad/s</param>
-      </state_interface>
-    </sensor>
+  </ros2_control>
+  <ros2_control name="IMU" type="sensor">
+    <hardware>
+      <plugin>mpu6050_hw/MPU6050HW</plugin>
+    </hardware>
+    <joint name="imu_joint">
+      <state_interface name="orientation.x"/>
+      <state_interface name="orientation.y"/>
+      <state_interface name="orientation.z"/>
+      <state_interface name="orientation.w"/>
+      <state_interface name="angular_velocity.x"/>
+      <state_interface name="angular_velocity.y"/>
+      <state_interface name="angular_velocity.z"/>
+      <state_interface name="linear_acceleration.x"/>
+      <state_interface name="linear_acceleration.y"/>
+      <state_interface name="linear_acceleration.z"/>
+    </joint>
   </ros2_control>
 </robot>

File: src/robot/robot_desc/urdf/four_wheel_chassis.xacro (robot description, xacro)
@@ -135,5 +135,5 @@
     </collision>
   </link>
-  <joint name="imu_joint" type="fixed">
+  <joint name="imu_joint" type="continuous">
     <parent link="base_link"/>
     <child link="imu"/>

Commit message: add rasp ubuntu

File: src/robot/robot_car_mecanum/urdf/robot_car.xacro (robot description, xacro)
@@ -1,26 +1,8 @@
 <?xml version="1.0" encoding="UTF-8"?>
 <robot name="robot_car_mecanum" xmlns:xacro="http://www.ros.org/wiki/xacro">
-  <!-- XML声明定义了文档使用的XML版本和UTF-8字符编码[1,3](@ref) -->
-  <!-- 参数使用仿真 -->
-  <xacro:arg name='use_gazebo' default='false'/>
-  <!-- 包含模型 -->
   <xacro:include filename="$(find robot_desc)/urdf/four_wheel_chassis.xacro"/>
-  <xacro:if value='$(arg use_gazebo)'>
-    <gazebo>
-      <plugin filename="gz_ros2_control-system" name="gz_ros2_control::GazeboSimROS2ControlPlugin">
-        <parameters>$(find robot_car_mecanum)/config/controllers.yaml</parameters>
-      </plugin>
-    </gazebo>
-  </xacro:if>
   <ros2_control name="mecanum_wheels_chassis" type="system">
     <hardware>
-      <xacro:if value="$(arg use_gazebo)">
-        <plugin>gz_ros2_control/GazeboSimSystem</plugin>
-      </xacro:if>
-      <xacro:unless value="$(arg use_gazebo)">
-        <plugin>four_wheel_chassis_hw/FourWheelChassisHW</plugin>
-        <!-- <plugin>mock_components/GenericSystem</plugin>
-        <param name="calculate_dynamics">true</param> -->
-      </xacro:unless>
+      <plugin>mecanum_wheel_chassis_hw/MecanumWheelChassisHW</plugin>
     </hardware>
     <joint name="left_front_wheel_joint">
@@ -48,10 +30,11 @@
     <hardware>
       <plugin>mpu6050_hw/MPU6050HW</plugin>
+      <param name="i2c_file_name">/dev/i2c-1</param>
     </hardware>
-    <joint name="imu_joint">
+    <sensor name="mpu6050">
+      <state_interface name="orientation.w"/>
       <state_interface name="orientation.x"/>
       <state_interface name="orientation.y"/>
       <state_interface name="orientation.z"/>
-      <state_interface name="orientation.w"/>
       <state_interface name="angular_velocity.x"/>
       <state_interface name="angular_velocity.y"/>
@@ -60,5 +43,5 @@
       <state_interface name="linear_acceleration.y"/>
       <state_interface name="linear_acceleration.z"/>
-    </joint>
+    </sensor>
   </ros2_control>
 </robot>

File: src/robot/robot_desc/urdf/four_wheel_chassis.xacro (robot description, xacro)
@@ -135,5 +135,5 @@
     </collision>
   </link>
-  <joint name="imu_joint" type="continuous">
+  <joint name="imu_joint" type="fixed">
     <parent link="base_link"/>
     <child link="imu"/>
