Commit message: base v2.0

File: src/robot_bringup/robot_car_mecanum/urdf/robot_car.xacro (robot description, xacro)
@@ -5,16 +5,17 @@
     <hardware>
       <plugin>mecanum_wheel_chassis_hw/MecanumWheelChassisHW</plugin>
-      <param name="use_topic">true</param>
       <param name="serial_port">/dev/ttyUSB0</param>
       <param name="baud_rate">115200</param>
-      <param name="encoder_ppr">255.0</param>
+      <param name="encoder_ppr">210.0</param>
       <param name="wheel_radius">0.03</param>
       <param name="gear_ratio">1</param>
-      <param name="max_pwm">255</param>
-      <param name="min_pwm">-255</param>
+      <param name="max_pwm">200</param>
+      <param name="min_pwm">10</param>
       <param name="lf_max_speed">10.0</param><!-- rad/s-->
       <param name="rf_max_speed">10.0</param>
       <param name="lr_max_speed">10.0</param>
       <param name="rr_max_speed">10.0</param>
+      <param name="use_server">true</param>
+      <param name="use_topic">true</param>
     </hardware>
     <joint name="left_front_wheel_joint">

File: src/robot_desc/urdf/four_wheel_chassis.xacro (robot description, xacro)
@@ -4,21 +4,37 @@
   <!-- ========================= 属性常量 ========================= -->
   <xacro:property name="PI" value="3.1415926535897931"/>
-  <xacro:property name="base_length"  value="0.26"/>
-  <xacro:property name="base_width"   value="0.16"/>
-  <xacro:property name="base_height"  value="0.04"/>
-  <xacro:property name="base_mass"    value="2.0"/>
+  <xacro:property name="base_length"  value="0.36"/>
+  <xacro:property name="base_width"   value="0.28"/>
+  <xacro:property name="base_height"  value="0.01"/>
+  <xacro:property name="base_mass"    value="2.8"/>
   <xacro:property name="wheel_radius" value="0.03"/>
   <xacro:property name="wheel_length" value="0.03"/>
-  <xacro:property name="wheel_mass"   value="0.5"/>
-  <xacro:property name="wheel_x" value="0.09"/>
-  <xacro:property name="wheel_y" value="0.11"/>
-  <xacro:property name="wheel_z" value="0.02"/>
+  <xacro:property name="wheel_mass"   value="0.09"/>
+  <xacro:property name="wheel_offset_x" value="0.15"/>
+  <xacro:property name="wheel_offset_y" value="0.17"/>
+  <xacro:property name="wheel_offset_z" value="0.04"/>
+  <xacro:property name="lidar_length" value="0.04"/>
+  <xacro:property name="lidar_radius" value="0.03"/>
+  <xacro:property name="lidar_mass" value="0.1"/>
+  <xacro:property name="lidar_offset_x" value="0.01"/>
+  <xacro:property name="lidar_offset_y" value="-0.05"/>
+  <xacro:property name="lidar_offset_z" value="0.115"/>
+  <xacro:property name="imu_width" value="0.02"/>
+  <xacro:property name="imu_length" value="0.02"/>
+  <xacro:property name="imu_height" value="0.02"/>
+  <xacro:property name="imu_mass" value="0.01"/>
+  <xacro:property name="imu_offset_x" value="0.0"/>
+  <xacro:property name="imu_offset_y" value="0.0"/>
+  <xacro:property name="imu_offset_z" value="0.005"/>
   <!-- 颜色 -->
   <xacro:property name="base_color" value="0 0.2 0.8 0.5"/>
   <xacro:property name="wheel_color" value="0 0 0 1"/>
+  <xacro:property name="lidar_color" value="0.5 0 0 1"/>
+  <xacro:property name="imu_color" value="0.5 0.5 0.5 1"/>
+  <!-- ========================= 材质宏 ========================= -->
   <material name="blue"><color rgba="${base_color}"/></material>
   <material name="black"><color rgba="${wheel_color}"/></material>
-  <material name="red"><color rgba="0.5 0 0 1"/></material>
-  <material name="gray"><color rgba="0.5 0.5 0.5 1"/></material>
+  <material name="red"><color rgba="${lidar_color}"/></material>
+  <material name="gray"><color rgba="${imu_color}"/></material>
   <!-- ========================= 惯性宏 ========================= -->
   <xacro:macro name="box_inertia" params="mass x y z">
@@ -64,5 +80,5 @@
     <parent link="base_footprint"/>
     <child link="base_link"/>
-    <origin xyz="0.0 0.0 0.04" rpy="0.0 0.0 0.0"/>
+    <origin xyz="0.0 0.0 0.07" rpy="0.0 0.0 0.0"/>
   </joint>
   <link name="base_link">
@@ -77,39 +93,39 @@
   </link>
   <!-- 四麦轮 -->
-  <xacro:create_wheel name="left_front"  xyz="${wheel_x}  ${wheel_y} -${wheel_z/2}"/>
-  <xacro:create_wheel name="right_front" xyz="${wheel_x} -${wheel_y} -${wheel_z/2}"/>
-  <xacro:create_wheel name="left_rear"   xyz="-${wheel_x}  ${wheel_y} -${wheel_z/2}"/>
-  <xacro:create_wheel name="right_rear"  xyz="-${wheel_x} -${wheel_y} -${wheel_z/2}"/>
+  <xacro:create_wheel name="left_front"  xyz="${wheel_offset_x}  ${wheel_offset_y} -${wheel_offset_z}"/>
+  <xacro:create_wheel name="right_front" xyz="${wheel_offset_x} -${wheel_offset_y} -${wheel_offset_z}"/>
+  <xacro:create_wheel name="left_rear"   xyz="-${wheel_offset_x}  ${wheel_offset_y} -${wheel_offset_z}"/>
+  <xacro:create_wheel name="right_rear"  xyz="-${wheel_offset_x} -${wheel_offset_y} -${wheel_offset_z}"/>
   <!-- 激光 -->
   <link name="laser_frame">
     <visual>
-      <geometry><cylinder radius="0.03" length="0.04"/></geometry>
+      <geometry><cylinder radius="${lidar_radius}" length="${lidar_length}"/></geometry>
       <material name="red"/>
     </visual>
     <collision>
-      <geometry><cylinder radius="0.03" length="0.04"/></geometry>
+      <geometry><cylinder radius="${lidar_radius}" length="${lidar_length}"/></geometry>
     </collision>
-    <xacro:cyl_inertia mass="0.1" r="0.03" h="0.04"/>
+    <xacro:cyl_inertia mass="${lidar_mass}" r="${lidar_radius}" h="${lidar_length}"/>
   </link>
   <joint name="laser_joint" type="fixed">
     <parent link="base_link"/>
     <child link="laser_frame"/>
-    <origin xyz="0 0 0.05" rpy="0 0 0"/>
+    <origin xyz="${lidar_offset_x} ${lidar_offset_y} ${lidar_offset_z}" rpy="0 0 0"/>
   </joint>
   <!-- IMU -->
   <link name="imu_link">
     <visual>
-      <geometry><box size="0.02 0.02 0.001"/></geometry>
+      <geometry><box size="${imu_width} ${imu_height} ${imu_length}"/></geometry>
       <material name="gray"/>
     </visual>
     <collision>
-      <geometry><box size="0.02 0.02 0.001"/></geometry>
+      <geometry><box size="${imu_width} ${imu_height} ${imu_length}"/></geometry>
     </collision>
-    <xacro:box_inertia mass="0.02" x="0.02" y="0.02" z="0.001"/>
+    <xacro:box_inertia mass="${imu_mass}" x="${imu_width}" y="${imu_height}" z="${imu_length}"/>
   </link>
   <joint name="imu_joint" type="fixed">
     <parent link="base_link"/>
     <child link="imu_link"/>
-    <origin xyz="0.045 0.06 0.025" rpy="0 0 0"/>
+    <origin xyz="${imu_offset_x} ${imu_offset_y} ${imu_offset_z}" rpy="0 0 0"/>
   </joint>
 </robot>
