Commit message: failure but save

File: src/robot_bringup/robot_car_mecanum/urdf/robot_car_voice.xacro (robot description, xacro)
@@ -1,5 +1,5 @@
 <?xml version="1.0" encoding="UTF-8"?>
 <robot name="robot_car_mecanum" xmlns:xacro="http://www.ros.org/wiki/xacro">
-  <xacro:include filename="$(find robot_desc)/urdf/four_wheel_chassis.xacro"/>
+  <xacro:include filename="$(find robot_desc)/urdf/four_wheel_chassis_voice.xacro"/>
   <xacro:include filename="$(find robot_car_mecanum)/urdf/robot_ros2_control.xacro"/>
 </robot>

File: src/robot_desc/urdf/four_wheel_chassis_voice.xacro (robot description, xacro)
@@ -2,20 +2,20 @@
 <robot name="four_wheel_chassis"
        xmlns:xacro="http://www.ros.org/wiki/xacro">
-  <xacro:property name="base_length"  value="0.36"/>
-  <xacro:property name="base_width"   value="0.28"/>
+  <xacro:property name="base_length"  value="0.44"/>
+  <xacro:property name="base_width"   value="0.40"/>
   <xacro:property name="base_height"  value="0.01"/>
-  <xacro:property name="base_mass"    value="2.8"/>
+  <xacro:property name="base_mass"    value="5.8"/>
   <xacro:property name="wheel_radius" value="0.03"/>
   <xacro:property name="wheel_length" value="0.03"/>
-  <xacro:property name="wheel_mass"   value="0.09"/>
-  <xacro:property name="wheel_offset_x" value="0.175"/>
-  <xacro:property name="wheel_offset_y" value="0.15"/>
+  <xacro:property name="wheel_mass"   value="0.1"/>
+  <xacro:property name="wheel_offset_x" value="0.19"/>
+  <xacro:property name="wheel_offset_y" value="0.185"/>
   <xacro:property name="wheel_offset_z" value="0.04"/>
   <xacro:property name="lidar_length" value="0.04"/>
   <xacro:property name="lidar_radius" value="0.03"/>
   <xacro:property name="lidar_mass" value="0.1"/>
-  <xacro:property name="lidar_offset_x" value="0.0"/>
+  <xacro:property name="lidar_offset_x" value="0.15"/>
   <xacro:property name="lidar_offset_y" value="0.0"/>
-  <xacro:property name="lidar_offset_z" value="0.115"/>
+  <xacro:property name="lidar_offset_z" value="0.12"/>
   <xacro:property name="imu_width" value="0.02"/>
   <xacro:property name="imu_length" value="0.02"/>
@@ -25,11 +25,4 @@
   <xacro:property name="imu_offset_y" value="0.0"/>
   <xacro:property name="imu_offset_z" value="0.01"/>
-  <xacro:property name="camera_width" value="0.04"/>
-  <xacro:property name="camera_length" value="0.12"/>
-  <xacro:property name="camera_height" value="0.04"/>
-  <xacro:property name="camera_mass" value="0.1"/>
-  <xacro:property name="camera_offset_x" value="0.1"/>
-  <xacro:property name="camera_offset_y" value="0.0"/>
-  <xacro:property name="camera_offset_z" value="0.05"/>
   <!-- ========================= 包含 ========================= -->
   <xacro:include filename="$(find robot_desc)/urdf/robot.xacro"/>
@@ -89,19 +82,3 @@
     <origin xyz="${imu_offset_x} ${imu_offset_y} ${imu_offset_z}" rpy="0 0 0"/>
   </joint>
-  <!-- Camera -->
-  <link name='camera_link'>
-      <visual>
-      <geometry><box size="${camera_width} ${camera_length} ${camera_height}"/></geometry>
-      <material name="gray"/>
-    </visual>
-    <collision>
-      <geometry><box size="${camera_width} ${camera_length} ${camera_height}"/></geometry>
-    </collision>
-    <xacro:box_inertia mass="${camera_mass}" x="${camera_width}" y="${camera_length}" z="${camera_height}"/>
-  </link>
-  <joint name="camera_joint" type="fixed">
-    <parent link="base_link"/>
-    <child link="camera_link"/>
-    <origin xyz="${camera_offset_x} ${camera_offset_y} ${camera_offset_z}" rpy="0 0 0"/>
-  </joint>
 </robot>
