Commit message: add lidar and position tracking controller

File: src/robot_desc/urdf/four_wheel_chassis.xacro (robot description, xacro)
@@ -22,5 +22,5 @@
   <xacro:property name="imu_width" value="0.02"/>
   <xacro:property name="imu_length" value="0.02"/>
-  <xacro:property name="imu_height" value="0.02"/>
+  <xacro:property name="imu_height" value="0.01"/>
   <xacro:property name="imu_mass" value="0.01"/>
   <xacro:property name="imu_offset_x" value="0.0"/>
